File: Development Board/Simulate-StackIntegration.sch (KiCad schematic (older format))
At the start: 2 parts

Commit message: Q-PACE Devboard V0
This should complete the KiCad Schematic and PCB files. Parts should be in FSI inventory.
Parts:
- J?: symbol conn:Conn_02x20_Odd_Even -> QPACE-DevelopmentBoard-rescue:Conn_02x20_Odd_Even-conn
- J?: symbol conn:Conn_02x12_Odd_Even -> QPACE-DevelopmentBoard-rescue:Conn_02x12_Odd_Even-conn
Changed lines of the file:
@@
 $Descr A4 11693 8268
 encoding utf-8
-Sheet 11 13
+Sheet 11 9
 Title ""
 Date ""
@@
 $EndDescr
 $Comp
-L conn:Conn_02x20_Odd_Even J?
+L QPACE-DevelopmentBoard-rescue:Conn_02x20_Odd_Even-conn J?
 U 1 1 5C88F6AB
 P 3700 4500
@@
 EN_Pi_Mux
 $Comp
-L conn:Conn_02x12_Odd_Even J?
+L QPACE-DevelopmentBoard-rescue:Conn_02x12_Odd_Even-conn J?
 U 1 1 5C88F6E5
 P 5800 4550
