File: Development Board/StatusLEDs.sch (KiCad schematic (older format))
At the start: 18 parts

Commit message: Q-PACE Devboard V0
This should complete the KiCad Schematic and PCB files. Parts should be in FSI inventory.
Parts:
- D? (x6): symbol device:LED -> QPACE-DevelopmentBoard-rescue:LED-device
- R? (x6): symbol device:R -> QPACE-DevelopmentBoard-rescue:R-device
Changed lines of the file:
@@
 $Descr A4 11693 8268
 encoding utf-8
-Sheet 13 13
+Sheet 13 9
 Title ""
 Date ""
@@
 $EndComp
 $Comp
-L device:R R?
+L QPACE-DevelopmentBoard-rescue:R-device R?
 U 1 1 5C946C7C
 P 3500 3150
@@
 $EndComp
 $Comp
-L device:R R?
+L QPACE-DevelopmentBoard-rescue:R-device R?
 U 1 1 5C946C83
 P 3500 4850
@@
 $EndComp
 $Comp
-L device:R R?
+L QPACE-DevelopmentBoard-rescue:R-device R?
 U 1 1 5C94C446
 P 5250 3200
@@
 $EndComp
 $Comp
-L device:R R?
+L QPACE-DevelopmentBoard-rescue:R-device R?
 U 1 1 5C94C44C
 P 5250 4850
@@
 UART_TX_CCDR
 $Comp
-L device:LED D?
+L QPACE-DevelopmentBoard-rescue:LED-device D?
 U 1 1 5C94C7BC
 P 3500 2850
@@
 $EndComp
 $Comp
-L device:LED D?
+L QPACE-DevelopmentBoard-rescue:LED-device D?
 U 1 1 5C94C852
 P 5250 2900
@@
 $EndComp
 $Comp
-L device:LED D?
+L QPACE-DevelopmentBoard-rescue:LED-device D?
 U 1 1 5C94C8FE
 P 5250 4550
@@
 $EndComp
 $Comp
-L device:LED D?
+L QPACE-DevelopmentBoard-rescue:LED-device D?
 U 1 1 5C94C952
 P 3500 4550
@@
 $EndComp
 $Comp
-L device:R R?
+L QPACE-DevelopmentBoard-rescue:R-device R?
 U 1 1 5C958B6F
 P 6800 3200
@@
 3V3_PGood
 $Comp
-L device:LED D?
+L QPACE-DevelopmentBoard-rescue:LED-device D?
 U 1 1 5C958B82
 P 6800 2900
@@
 $EndComp
 $Comp
-L device:R R?
+L QPACE-DevelopmentBoard-rescue:R-device R?
 U 1 1 5C958C4D
 P 6800 4800
@@
 5V_PGood
 $Comp
-L device:LED D?
+L QPACE-DevelopmentBoard-rescue:LED-device D?
 U 1 1 5C958C60
 P 6800 4500
