File: Development Board/QPACE-DevelopmentBoard.sch (KiCad schematic (older format))
At the start: 0 parts

Commit message: main sheets created
Parts:
- added D? (x2): D_Schottky, symbol Device:D_Schottky
- added F?: Polyfuse, symbol Device:Polyfuse
- added J?: USB_B_Micro, symbol Connector:USB_B_Micro
- added J?: Power Jack_opt, symbol Connector_Generic:Conn_01x02
Connections:
- net labels added: +3.3V, +5V, GND, USB_5V, USB_D+, USB_D-
- wire segments 0 -> 55
- no-connect marks 0 -> 2

Commit message: added FTDI
Parts:
- added J?: CCDR_External, symbol conn:Conn_01x04
- added J?: RF_External, symbol conn:Conn_01x04
- added SW? (x4): SW_DPDT_x2, symbol Switch:SW_DPDT_x2
Connections:
- wire segments 55 -> 84
Other:
- note added: "simluate RF"
Changed lines of the file:
@@
 $Descr A4 11693 8268
 encoding utf-8
-Sheet 1 9
+Sheet 1 10
 Title "Raspberry Pi HAT"
 Date ""
@@
 $EndDescr
 $Sheet
-S 5700 3550 550  550
+S 9200 3750 600  550
 U 5C7F607C
 F0 "Simulate-CCDR" 50
 F1 "Simulate-CCDR.sch" 50
-F2 "USB_D+" I L 5700 3700 50
-F3 "USB_D-" I L 5700 3800 50
-F4 "UART_TX" I R 6250 3900 50
-F5 "UART_RX" I R 6250 4000 50
+F2 "UART_TX" I R 9800 4100 50
+F3 "UART_RX" I R 9800 4200 50
+F4 "COM_TX" I L 9200 3900 50
+F5 "COM_RX" I L 9200 4000 50
 $EndSheet
 $Sheet
@@
 Wire Wire Line
 	5050 2150 5700 2150
-$Sheet
-S 5700 2650 900  400
-U 5C955249
-F0 "Simluate-RF" 50
-F1 "Simluate-RF.sch" 50
-F2 "USB_D+" I L 5700 2800 50
-F3 "USB_D-" I L 5700 2900 50
-F4 "UART_TX" I R 6600 2800 50
-F5 "UART_RX" I R 6600 2900 50
-$EndSheet
-Wire Wire Line
-	5700 3700 5200 3700
 Wire Wire Line
 	5200 3700 5200 3000
@@
 Wire Wire Line
 	5100 3100 5100 3800
-Wire Wire Line
-	5100 3800 5700 3800
 $Sheet
 S 1000 1400 750  300
@@
 	2150 3600 2350 3600
 Wire Wire Line
-	4700 2800 5700 2800
-Wire Wire Line
-	4700 2900 5700 2900
-Wire Wire Line
 	3750 2600 1900 2600
 Wire Wire Line
@@
 	1850 2700 3750 2700
 Wire Wire Line
-	6600 2800 7050 2800
-Wire Wire Line
-	7050 2800 7050 1000
-Wire Wire Line
-	7050 1000 3100 1000
-Wire Wire Line
 	3150 1600 3100 1600
 Wire Wire Line
@@
 	3000 1700 3000 900
 Wire Wire Line
-	3000 900  7150 900
-Wire Wire Line
-	7150 900  7150 2900
-Wire Wire Line
-	7150 2900 6600 2900
+	9950 900  9950 2600
 Wire Wire Line
 	3150 1800 2900 1800
@@
 	2900 1800 2900 800
 Wire Wire Line
-	2900 800  7250 800
-Wire Wire Line
-	7250 800  7250 3900
-Wire Wire Line
-	7250 3900 6250 3900
-Wire Wire Line
-	6250 4000 7350 4000
-Wire Wire Line
-	7350 4000 7350 700
-Wire Wire Line
-	7350 700  2800 700
-Wire Wire Line
 	2800 700  2800 1900
 Wire Wire Line
 	2800 1900 3150 1900
+$Comp
+L Switch:SW_DPDT_x2 SW?
+U 1 1 5C832814
+P 7400 3550
+F 0 "SW?" H 7400 3835 50  0000 C CNN
+F 1 "SW_DPDT_x2" H 7400 3744 50  0000 C CNN
+F 2 "" H 7400 3550 50  0001 C CNN
+F 3 "" H 7400 3550 50  0001 C CNN
+	1    7400 3550
+	1    0    0    -1
+$EndComp
+$Comp
+L Switch:SW_DPDT_x2 SW?
+U 2 1 5C832863
+P 7400 4100
+F 0 "SW?" H 7400 4385 50  0000 C CNN
+F 1 "SW_DPDT_x2" H 7400 4294 50  0000 C CNN
+F 2 "" H 7400 4100 50  0001 C CNN
+F 3 "" H 7400 4100 50  0001 C CNN
+	2    7400 4100
+	1    0    0    -1
+$EndComp
+$Sheet
+S 5800 2700 900  300
+U 5C83EBD8
+F0 "FTDI_0" 50
+F1 "FTDI.sch" 50
+F2 "USB_D+" I L 5800 2800 50
+F3 "USB_D-" I L 5800 2900 50
+F4 "UART_TX" I R 6700 2800 50
+F5 "UART_RX" I R 6700 2900 50
+$EndSheet
+$Sheet
+S 5800 3600 900  300
+U 5C84505A
+F0 "FTDI_1" 50
+F1 "FTDI.sch" 50
+F2 "USB_D+" I L 5800 3700 50
+F3 "USB_D-" I L 5800 3800 50
+F4 "UART_TX" I R 6700 3700 50
+F5 "UART_RX" I R 6700 3800 50
+$EndSheet
+Wire Wire Line
+	10050 800  10050 4100
+Wire Wire Line
+	10150 4200 9800 4200
+Wire Wire Line
+	10150 700  10150 4200
+Wire Wire Line
+	9800 4100 10050 4100
+$Comp
+L conn:Conn_01x04 J?
+U 1 1 5C8563BD
+P 8950 4300
+F 0 "J?" H 9030 4292 50  0000 L CNN
+F 1 "CCDR_External" H 9030 4201 50  0000 L CNN
+F 2 "" H 8950 4300 50  0001 C CNN
+F 3 "~" H 8950 4300 50  0001 C CNN
+	1    8950 4300
+	1    0    0    -1
+$EndComp
+Wire Wire Line
+	5800 3700 5200 3700
+Wire Wire Line
+	5100 3800 5800 3800
+Wire Wire Line
+	4700 2800 5800 2800
+Wire Wire Line
+	4700 2900 5800 2900
+$Comp
+L Switch:SW_DPDT_x2 SW?
+U 1 1 5C882577
+P 7400 2600
+F 0 "SW?" H 7400 2885 50  0000 C CNN
+F 1 "SW_DPDT_x2" H 7400 2794 50  0000 C CNN
+F 2 "" H 7400 2600 50  0001 C CNN
+F 3 "" H 7400 2600 50  0001 C CNN
+	1    7400 2600
+	1    0    0    -1
+$EndComp
+$Comp
+L Switch:SW_DPDT_x2 SW?
+U 2 1 5C88257D
+P 7400 3100
+F 0 "SW?" H 7400 3385 50  0000 C CNN
+F 1 "SW_DPDT_x2" H 7400 3294 50  0000 C CNN
+F 2 "" H 7400 3100 50  0001 C CNN
+F 3 "" H 7400 3100 50  0001 C CNN
+	2    7400 3100
+	1    0    0    -1
+$EndComp
+Wire Wire Line
+	7200 3550 7000 3550
+Wire Wire Line
+	7000 3550 7000 3700
+Wire Wire Line
+	6700 3700 7000 3700
+Wire Wire Line
+	7200 4100 7100 4100
+Wire Wire Line
+	7100 4100 7100 3800
+Wire Wire Line
+	6700 3800 7100 3800
+Wire Wire Line
+	7200 3100 7050 3100
+Wire Wire Line
+	7050 3100 7050 2900
+Wire Wire Line
+	7050 2900 6700 2900
+Wire Wire Line
+	6700 2800 7050 2800
+Wire Wire Line
+	7050 2800 7050 2600
+Wire Wire Line
+	7050 2600 7200 2600
+Wire Wire Line
+	7600 3000 7800 3000
+Wire Wire Line
+	7800 3000 7800 2600
+$Comp
+L conn:Conn_01x04 J?
+U 1 1 5C8928CF
+P 9000 3100
+F 0 "J?" H 9079 3092 50  0000 L CNN
+F 1 "RF_External" H 9079 3001 50  0000 L CNN
+F 2 "" H 9000 3100 50  0001 C CNN
+F 3 "~" H 9000 3100 50  0001 C CNN
+	1    9000 3100
+	1    0    0    -1
+$EndComp
+Wire Wire Line
+	9200 3900 8200 3900
+Wire Wire Line
+	8200 3900 8200 3450
+Wire Wire Line
+	8200 3450 7600 3450
+Wire Wire Line
+	7600 4000 9200 4000
+Wire Wire Line
+	7900 4400 7900 3650
+Wire Wire Line
+	7900 3650 7600 3650
+Wire Wire Line
+	7800 4200 7800 4500
+Wire Wire Line
+	7600 4200 7800 4200
+$Comp
+L power:GND #PWR?
+U 1 1 5C89E7CC
+P 8800 3100
+F 0 "#PWR?" H 8800 2850 50  0001 C CNN
+F 1 "GND" V 8805 2972 50  0000 R CNN
+F 2 "" H 8800 3100 50  0001 C CNN
+F 3 "" H 8800 3100 50  0001 C CNN
+	1    8800 3100
+	0    1    1    0
+$EndComp
+Wire Wire Line
+	9850 1000 9850 2500
+Wire Wire Line
+	7800 2600 9950 2600
+Wire Wire Line
+	7700 3200 7700 2700
+Wire Wire Line
+	7700 2700 7600 2700
+Wire Wire Line
+	7600 3200 7600 3300
+$Comp
+L power:GND #PWR?
+U 1 1 5C8A03B3
+P 8750 4300
+F 0 "#PWR?" H 8750 4050 50  0001 C CNN
+F 1 "GND" V 8750 4100 50  0000 C CNN
+F 2 "" H 8750 4300 50  0001 C CNN
+F 3 "" H 8750 4300 50  0001 C CNN
+	1    8750 4300
+	0    1    1    0
+$EndComp
+Wire Wire Line
+	7700 3200 8800 3200
+Wire Wire Line
+	7600 3300 8800 3300
+Wire Wire Line
+	7900 4400 8750 4400
+Wire Wire Line
+	7800 4500 8750 4500
+$Comp
+L power:+5V #PWR?
+U 1 1 5C8D1FFE
+P 8750 4200
+F 0 "#PWR?" H 8750 4050 50  0001 C CNN
+F 1 "+5V" H 8765 4373 50  0000 C CNN
+F 2 "" H 8750 4200 50  0001 C CNN
+F 3 "" H 8750 4200 50  0001 C CNN
+	1    8750 4200
+	1    0    0    -1
+$EndComp
+$Comp
+L power:+5V #PWR?
+U 1 1 5C8D2051
+P 8800 3000
+F 0 "#PWR?" H 8800 2850 50  0001 C CNN
+F 1 "+5V" H 8815 3173 50  0000 C CNN
+F 2 "" H 8800 3000 50  0001 C CNN
+F 3 "" H 8800 3000 50  0001 C CNN
+	1    8800 3000
+	1    0    0    -1
+$EndComp
+Wire Wire Line
+	7600 2500 9850 2500
+Text Notes 6400 2600 0    50   ~ 0
+simluate RF
+Wire Wire Line
+	2800 700  10150 700
+Wire Wire Line
+	2900 800  10050 800
+Wire Wire Line
+	3000 900  9950 900
+Wire Wire Line
+	3100 1000 9850 1000
 $EndSCHEMATC

Commit message: added extra USB port, gyroscope, stack connector
Much more work needs to be done. almost all high level sheets are made
Parts:
- added C? (x2): 0.1uF, symbol device:C
- added D?: LED_Dual_AACC, symbol device:LED_Dual_AACC
- added J?: Avionics Stack Connector, symbol conn:Conn_02x20_Odd_Even
- added J?: I2C-BUS, symbol conn:Conn_01x02
- added J?: CCDR-ECR Connector, symbol conn:Conn_02x12_Odd_Even
- added J?: SWD, symbol conn:Conn_02x03_Odd_Even
- added J? (x2): USB_A, symbol conn:USB_A
- added R? (x2): 10k, symbol device:R
- added U?: BMG160, symbol QPACE-SchematicSymbols:BMG160
Connections:
- net labels added: 12V_Rail, 3V3_Rail, 5V_Rail, EN_12V-1, EN_12V-2, EN_5V-1, EN_5V-2, EN_LED, EN_Pi1_Pwr, EN_Pi2_Pwr, EN_Pi_Mux, EN_Solenoid1, EN_Solenoid2, EN_Solenoid3, EN_Stepper, EN_Stepper_A, EN_Stepper_B, I2C_SCL, I2C_SDA, Pi1_GPIO, Pi2_GPIO, UART_RX_Pi1, UART_RX_Pi2, UART_TX_Pi1, UART_TX_Pi2, Vbat
- wire segments 84 -> 143
- no-connect marks 2 -> 23
Other:
- note added: "GYROSCOPE onboard of CCDR \nI2C Comms"
- note added: "Use the "Avionics Stack Connector" to attach \nto the engineering model to test functionality"
- note added: "Use the "CCDR-ECR Connector" to attach \nto the Experiment Control/Regulator board \nto test ETC (experiment test cell) functionality"
- note added: "recommend using one of these \nports to connect an ethernet-USB \nconverter from Pi to this port."
- moved on the sheet: D?, J?

Commit message: added KISS description, UART-I2C chip
keep it simple, stupid. Goal is to create software development board for sub-system comms
Parts:
- removed D?: D_Schottky, symbol Device:D_Schottky
- removed F?: Polyfuse, symbol Device:Polyfuse
- removed J?: Avionics Stack Connector, symbol conn:Conn_02x20_Odd_Even
- removed J?: CCDR-ECR Connector, symbol conn:Conn_02x12_Odd_Even
Connections:
- net labels removed: 12V_Rail, 3V3_Rail, 5V_Rail, EN_12V-1, EN_12V-2, EN_5V-1, EN_5V-2, EN_LED, EN_Pi1_Pwr, EN_Pi2_Pwr, EN_Pi_Mux, EN_Solenoid1, EN_Solenoid2, EN_Solenoid3, EN_Stepper, EN_Stepper_A, EN_Stepper_B, Pi1_GPIO, Pi2_GPIO, UART_RX_Pi1, UART_RX_Pi2, UART_TX_Pi1, UART_TX_Pi2, Vbat
- wire segments 143 -> 128
- no-connect marks 23 -> 7
Other:
- note added: "Pi ethernet 2 USB adp."
- note added: "extra USB\n"
- note removed: "Use the "Avionics Stack Connector" to attach \nto the engineering model to test functionality"
- note removed: "Use the "CCDR-ECR Connector" to attach \nto the Experiment Control/Regulator board \nto test ETC (experiment test cell) functionality"
Changed lines of the file:
@@
 $Descr A4 11693 8268
 encoding utf-8
-Sheet 1 10
+Sheet 1 12
 Title "Raspberry Pi HAT"
 Date ""
@@
 Text Label 1150 2400 0    50   ~ 0
 USB_5V
-Wire Wire Line
-	1150 2400 1500 2400
-$Comp
-L Device:Polyfuse F?
-U 1 1 5C955A1A
-P 1650 2400
-F 0 "F?" V 1550 2350 50  0000 C CNN
-F 1 "Polyfuse" V 1750 2350 50  0000 C CNN
-F 2 "" H 1700 2200 50  0001 L CNN
-F 3 "~" H 1650 2400 50  0001 C CNN
-	1    1650 2400
-	0    1    1    0
-$EndComp
-$Comp
-L Device:D_Schottky D?
-U 1 1 5C955B19
-P 2050 2400
-F 0 "D?" H 2050 2184 50  0000 C CNN
-F 1 "D_Schottky" H 2050 2275 50  0000 C CNN
-F 2 "" H 2050 2400 50  0001 C CNN
-F 3 "~" H 2050 2400 50  0001 C CNN
-	1    2050 2400
-	-1   0    0    1
-$EndComp
-Wire Wire Line
-	1900 2400 1800 2400
 Text Label 1150 2600 0    50   ~ 0
 USB_D+
@@
 $EndSheet
 Wire Wire Line
-	10800 800  10800 4100
-Wire Wire Line
-	10900 4200 9800 4200
-Wire Wire Line
-	10900 700  10900 4200
-Wire Wire Line
-	9800 4100 10800 4100
+	10100 800  10100 4100
+Wire Wire Line
+	10200 4200 9800 4200
+Wire Wire Line
+	10200 700  10200 4200
+Wire Wire Line
+	9800 4100 10100 4100
 $Comp
 L conn:Conn_01x04 J?
@@
 simluate RF
 Wire Wire Line
-	2800 700  10900 700
-Wire Wire Line
-	2900 800  10800 800
+	2800 700  10200 700
+Wire Wire Line
+	2900 800  10100 800
 Wire Wire Line
 	3000 900  9950 900
 Wire Wire Line
 	3100 1000 9850 1000
-$Comp
-L conn:Conn_02x20_Odd_Even J?
-U 1 1 5C8E5364
-P 1600 6500
-F 0 "J?" H 1650 7617 50  0000 C CNN
-F 1 "Avionics Stack Connector" H 1650 7526 50  0000 C CNN
-F 2 "" H 1600 6500 50  0001 C CNN
-F 3 "~" H 1600 6500 50  0001 C CNN
-	1    1600 6500
-	1    0    0    -1
-$EndComp
-Text Label 1400 5600 2    50   ~ 0
-UART_TX_Pi2
-Text Label 1400 5700 2    50   ~ 0
-UART_RX_Pi2
-Text Label 1400 5800 2    50   ~ 0
-UART_TX_Pi1
-Text Label 1400 5900 2    50   ~ 0
-UART_RX_Pi1
-Text Label 1400 6000 2    50   ~ 0
-Pi1_GPIO
-Text Label 1400 6100 2    50   ~ 0
-I2C_SDA
-Text Label 1400 6200 2    50   ~ 0
-I2C_SCL
-Text Label 1400 6400 2    50   ~ 0
-EN_12V-1
-Text Label 1900 7500 0    50   ~ 0
-3V3_Rail
-Text Label 1900 7200 0    50   ~ 0
-Vbat
-Text Label 1900 7100 0    50   ~ 0
-Vbat
-Text Label 1400 7100 2    50   ~ 0
-Vbat
-Text Label 1400 7200 2    50   ~ 0
-Vbat
-Text Label 1400 7500 2    50   ~ 0
-5V_Rail
-Wire Wire Line
-	1400 7500 1400 7400
-Connection ~ 1400 7400
-Wire Wire Line
-	1400 7400 1400 7300
-Wire Wire Line
-	1900 7400 1900 7500
-Text Label 1900 7000 0    50   ~ 0
-EN_5V-2
-Text Label 1400 7000 2    50   ~ 0
-EN_5V-1
-NoConn ~ 1900 6900
-NoConn ~ 1400 6900
-$Comp
-L power:GND #PWR?
-U 1 1 5C8EFA47
-P 1900 6700
-F 0 "#PWR?" H 1900 6450 50  0001 C CNN
-F 1 "GND" V 1905 6572 50  0000 R CNN
-F 2 "" H 1900 6700 50  0001 C CNN
-F 3 "" H 1900 6700 50  0001 C CNN
-	1    1900 6700
-	0    -1   -1   0
-$EndComp
-$Comp
-L power:GND #PWR?
-U 1 1 5C8EFA95
-P 1400 6700
-F 0 "#PWR?" H 1400 6450 50  0001 C CNN
-F 1 "GND" V 1405 6572 50  0000 R CNN
-F 2 "" H 1400 6700 50  0001 C CNN
-F 3 "" H 1400 6700 50  0001 C CNN
-	1    1400 6700
-	0    1    1    0
-$EndComp
-Wire Wire Line
-	1900 6600 1900 6700
-Connection ~ 1900 6700
-Wire Wire Line
-	1900 6700 1900 6800
-Wire Wire Line
-	1400 6600 1400 6700
-Connection ~ 1400 6700
-Wire Wire Line
-	1400 6700 1400 6800
-Text Label 1900 6400 0    50   ~ 0
-EN_12V-2
-Text Label 1900 5700 0    50   ~ 0
-Pi2_GPIO
-Text Label 1900 5800 0    50   ~ 0
-EN_Pi1_Pwr
-Text Label 1900 5900 0    50   ~ 0
-EN_Pi2_Pwr
-NoConn ~ 1900 6000
-NoConn ~ 1900 6100
-NoConn ~ 1900 6200
-NoConn ~ 1900 6300
-Text Label 1400 6300 2    50   ~ 0
-12V_Rail
-NoConn ~ 1900 7300
-Text Label 1900 5600 0    50   ~ 0
-EN_Pi_Mux
 $Comp
 L conn:Conn_01x02 J?
@@
 Text Label 1650 4600 2    50   ~ 0
 I2C_SCL
-$Comp
-L conn:Conn_02x12_Odd_Even J?
-U 1 1 5C9104EC
-P 3700 6550
-F 0 "J?" H 3750 7267 50  0000 C CNN
-F 1 "CCDR-ECR Connector" H 3750 7176 50  0000 C CNN
-F 2 "" H 3700 6550 50  0001 C CNN
-F 3 "~" H 3700 6550 50  0001 C CNN
-	1    3700 6550
-	1    0    0    -1
-$EndComp
-$Comp
-L power:GND #PWR?
-U 1 1 5C910592
-P 3500 6050
-F 0 "#PWR?" H 3500 5800 50  0001 C CNN
-F 1 "GND" V 3505 5922 50  0000 R CNN
-F 2 "" H 3500 6050 50  0001 C CNN
-F 3 "" H 3500 6050 50  0001 C CNN
-	1    3500 6050
-	0    1    1    0
-$EndComp
-Wire Wire Line
-	3500 6050 3500 6150
-Connection ~ 3500 6150
-Wire Wire Line
-	3500 6150 3500 6250
-Connection ~ 3500 6250
-Wire Wire Line
-	3500 6250 3500 6350
-Connection ~ 3500 6050
-Wire Wire Line
-	4000 6050 4000 6150
-Connection ~ 4000 6150
-Wire Wire Line
-	4000 6150 4000 6250
-Connection ~ 4000 6250
-Wire Wire Line
-	4000 6250 4000 6350
-$Comp
-L power:GND #PWR?
-U 1 1 5C914FC2
-P 4000 6050
-F 0 "#PWR?" H 4000 5800 50  0001 C CNN
-F 1 "GND" V 4005 5922 50  0000 R CNN
-F 2 "" H 4000 6050 50  0001 C CNN
-F 3 "" H 4000 6050 50  0001 C CNN
-	1    4000 6050
-	0    -1   -1   0
-$EndComp
-Connection ~ 4000 6050
-Text Label 3500 6450 2    50   ~ 0
-EN_Solenoid2
-Text Label 3500 6550 2    50   ~ 0
-EN_Stepper
-Text Label 3500 6650 2    50   ~ 0
-EN_Stepper_A
-Text Label 3500 6750 2    50   ~ 0
-EN_Stepper_B
-NoConn ~ 3500 6850
-NoConn ~ 3500 6950
-NoConn ~ 3500 7050
-NoConn ~ 3500 7150
-NoConn ~ 4000 7150
-NoConn ~ 4000 7050
-NoConn ~ 4000 6950
-NoConn ~ 4000 6850
-NoConn ~ 4000 6750
-Text Label 4000 6450 0    50   ~ 0
-EN_Solenoid3
-Text Label 4000 6550 0    50   ~ 0
-EN_Solenoid1
-Text Label 4000 6650 0    50   ~ 0
-EN_LED
 $Comp
 L QPACE-SchematicSymbols:BMG160 U?
@@
 Wire Wire Line
 	2600 1550 2600 2400
-Wire Wire Line
-	2600 2400 2200 2400
 $Comp
 L device:LED_Dual_AACC D?
@@
 Wire Wire Line
 	5300 1900 4250 1900
-Text Notes 900  5100 0    50   ~ 0
-Use the "Avionics Stack Connector" to attach \nto the engineering model to test functionality
-Text Notes 3050 5700 0    50   ~ 0
-Use the "CCDR-ECR Connector" to attach \nto the Experiment Control/Regulator board \nto test ETC (experiment test cell) functionality
 Wire Wire Line
 	2150 3600 2350 3600
@@
 Text Notes 5750 4350 0    50   ~ 0
 recommend using one of these \nports to connect an ethernet-USB \nconverter from Pi to this port.
+$Sheet
+S 10300 750  500  450
+U 5C86F6E8
+F0 "QPACE_DevBoard-R0" 50
+F1 "QPACE_DevBoard-R0.sch" 50
+$EndSheet
+Text Notes 4100 4000 0    50   ~ 0
+Pi ethernet 2 USB adp.
+$Sheet
+S 2650 5600 800  650
+U 5C872C63
+F0 "Simulate-StackIntegration" 50
+F1 "Simulate-StackIntegration.sch" 50
+$EndSheet
+Wire Wire Line
+	1150 2400 2600 2400
+Text Notes 5700 4950 0    50   ~ 0
+extra USB\n
 $EndSCHEMATC

Commit message: reduced complexity
Parts:
- removed D?: LED_Dual_AACC, symbol device:LED_Dual_AACC
- removed J?: SWD, symbol conn:Conn_02x03_Odd_Even
- removed J? (x2): USB_A, symbol conn:USB_A
- added C?: 0.1uF, symbol device:C
- added J?: SWD_ext, symbol conn:Conn_01x06
- added R?: 10k, symbol device:R
- added SW?: SW_SPDT, symbol Switch:SW_SPDT
- added U?: TS5N412, symbol QPACE-SchematicSymbols:TS5N412
Connections:
- net labels added: NRST, NRST_ext, NRST_int, SWCLK, SWCLK_ext, SWCLK_int, SWDIO, SWDIO_ext, SWDIO_int, SWO, SWO_ext, SWO_int, UART_RX_CCDR, UART_RX_CCDR_ext, UART_RX_CCDR_int, UART_RX_RF, UART_RX_RF_ext, UART_RX_RF_int, UART_TX_CCDR, UART_TX_CCDR_ext, UART_TX_CCDR_int, UART_TX_RF, UART_TX_RF_ext, UART_TX_RF_int
- wire segments 128 -> 116
- no-connect marks 7 -> 5
Other:
- note removed: "Pi ethernet 2 USB adp."
- note removed: "extra USB\n"
- note removed: "recommend using one of these \nports to connect an ethernet-USB \nconverter from Pi to this port."
- moved on the sheet: C?, D?, J?, R?, SW?A, SW?B, U?

Commit message: Q-PACE Devboard V0
This should complete the KiCad Schematic and PCB files. Parts should be in FSI inventory.
Parts:
- removed C?: 0.1uF, symbol device:C
- removed J?: CCDR_External, symbol conn:Conn_01x04
- removed J?: I2C-BUS, symbol conn:Conn_01x02
- removed J?: USB_B_Micro, symbol Connector:USB_B_Micro
- removed J?: Power Jack_opt, symbol Connector_Generic:Conn_01x02
- removed R?: 10k, symbol device:R
- removed SW? (x4): SW_DPDT_x2, symbol Switch:SW_DPDT_x2
- removed SW?: SW_SPDT, symbol Switch:SW_SPDT
- removed U?: TS5N412, symbol QPACE-SchematicSymbols:TS5N412
- added D1, D3: D_Schottky, project_footprints:SOD-128, symbol Device:D_Schottky
- added J1: Barrel_Jack_Switch, TerminalBlocks_Phoenix:TerminalBlock_Phoenix_PT-3.5mm_2pol, symbol Connector:Barrel_Jack_Switch
- added J12: USB-Serial, Socket_Strips:Socket_Strip_Straight_1x03_Pitch2.54mm, symbol Connector_Generic:Conn_01x03
- added J2: 5Vin-USB, Socket_Strips:Socket_Strip_Straight_1x02_Pitch2.54mm, symbol Connector_Generic:Conn_01x02
- added J3, J4: Vin, project_footprints:Socket_Strip_Straight_1x02_Pitch15.24mm, symbol Connector_Generic:Conn_01x02
- added J6: WTC_I2C-BUS, Socket_Strips:Socket_Strip_Straight_1x03_Pitch2.54mm, symbol Connector_Generic:Conn_01x03
- added J7, J8: Vout, project_footprints:Socket_Strip_Straight_1x02_Pitch15.24mm, symbol Connector_Generic:Conn_01x02
- added J9: GPS, Socket_Strips:Socket_Strip_Straight_1x06_Pitch2.54mm, symbol Connector_Generic:Conn_01x06
- added R1: 100k, Resistors_SMD:R_0805, symbol QPACE-DevelopmentBoard-rescue:R-device
- added SW2: SW_SPDT, Socket_Strips:Socket_Strip_Straight_1x03_Pitch2.54mm, symbol Switch:SW_SPDT
- added TP1, TP2, TP3, TP4: TestPoint, Measurement_Points:Measurement_Point_Round-SMD-Pad_Small, symbol Connector:TestPoint
- C1, C2: renamed from C?; footprint (none) -> Capacitors_SMD:C_0805; symbol device:C -> QPACE-DevelopmentBoard-rescue:C-device
- D2: renamed from D?; footprint (none) -> project_footprints:SOD-128
- J10: renamed from J?; footprint (none) -> Socket_Strips:Socket_Strip_Straight_1x06_Pitch2.54mm; symbol conn:Conn_01x06 -> QPACE-DevelopmentBoard-rescue:Conn_01x06-conn
- J13: renamed from J?; footprint (none) -> Socket_Strips:Socket_Strip_Straight_1x04_Pitch2.54mm; symbol conn:Conn_01x04 -> QPACE-DevelopmentBoard-rescue:Conn_01x04-conn
- R2, R3: renamed from R?; footprint (none) -> Resistors_SMD:R_0805; symbol device:R -> QPACE-DevelopmentBoard-rescue:R-device
- U1: renamed from U?; footprint (none) -> project_footprints:LGA-12_2x2mm_Pitch0.5mm; symbol QPACE-SchematicSymbols:BMG160 -> QPACE-DevelopmentBoard-rescue:BMG160-QPACE-SchematicSymbols
Connections:
- net NRST_ext is gone; now on net NRST: J10.5 (Pin_5)
- net SWCLK_ext is gone; now on net SWDIO: J10.3 (Pin_3)
- net SWDIO_ext is gone; now on net SWCLK: J10.4 (Pin_4)
- net SWO_ext is gone; now on net SWO: J10.6 (Pin_6)
- net UART_RX_RF_ext is gone; now on net UART_RX_RF_int: J13.4 (Pin_4)
- net UART_TX_RF_ext is gone; now on net UART_TX_RF_int: J13.3 (Pin_3)
- net +3V3: now also J8.1 (Pin_1), J9.1 (Pin_1), R1.1, TP3.1
- net +5V: now also D3.1 (K), J4.1 (Pin_1), J9.2 (Pin_2), TP4.1
- net GND: now also J1.2, J1.3, J12.3 (Pin_3), J2.2 (Pin_2), J3.2 (Pin_2), J4.2 (Pin_2), J6.3 (Pin_3), J7.2 (Pin_2), J8.2 (Pin_2), J9.3 (Pin_3)
- net I2C_SCL: now also J6.2 (Pin_2)
- net I2C_SDA: now also J6.1 (Pin_1)
- net UART_RX_CCDR: now also J12.2 (Pin_2)
- net UART_TX_CCDR: now also J12.1 (Pin_1)
- net BuckBoost-5Vout/5Vout: no longer names the net of D2.2 (A)
- net BuckBoost-5Vout/5Vout: now also J7.1 (Pin_1)
- new net: D3.2 (A), J2.1 (Pin_1), TP2.1
- new net: D1.1 (K), J3.1 (Pin_1)
- new net: D1.2 (A), J1.1, TP1.1
- new net: R1.2, SW2.2 (B)
- new net En_PiPwr: SW2.1 (A)
- new net GPS_EN: J9.6 (Pin_6)
- new net GPS_RX: J9.5 (Pin_5)
- new net GPS_TX: J9.4 (Pin_4)
- no-connect marks 5 -> 4
Other:
- note added: "------------------------------------------------------------------------------------\nThe purpose of QPACE Devboard Revision 0 is ONLY to allow the software team to quickly \ndevelop the comms between systems. Later revisions may incorporate adding features like stack integration and sub-system testing/analysis.\n------------------------------------------------------------------------------------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"
- moved on the sheet: C1, C2, J10, J13, R2, R3, U1
