File: Development Board/QPACE-DevelopmentBoard.sch (KiCad schematic (older format))
At the start: 25 parts, among them J1 Barrel_Jack_Switch, J10 SWD_ext, J12 USB-Serial, J13 RF_External, J2 5Vin-USB, J3 Vin, J4 Vin, J6 WTC_I2C-BUS, J7 Vout, J8 Vout, J9 GPS, SW2 SW_SPDT, U1 BMG160

Commit message: added silk screen, organized pins
Parts:
- removed J12: USB-Serial, Socket_Strips:Socket_Strip_Straight_1x03_Pitch2.54mm, symbol Connector_Generic:Conn_01x03
- added J5: RPi_COMPort, Socket_Strips:Socket_Strip_Straight_1x04_Pitch2.54mm, symbol QPACE-DevelopmentBoard-rescue:Conn_01x04-conn
Connections:
- net +5V: now also J5.1 (Pin_1)
- net GND: now also J5.2 (Pin_2)
- net UART_RX_CCDR: now also J5.4 (Pin_4)
- net UART_TX_CCDR: now also J5.3 (Pin_3)
Changed lines of the file:
@@
 Connection ~ 3100 3550
-$Comp
-L Connector_Generic:Conn_01x03 J12
-U 1 1 5CBED299
-P 8650 6000
-F 0 "J12" H 8650 6200 50  0000 C CNN
-F 1 "USB-Serial" H 8600 5750 50  0000 C CNN
-F 2 "Socket_Strips:Socket_Strip_Straight_1x03_Pitch2.54mm" H 8650 6000 50  0001 C CNN
-F 3 "~" H 8650 6000 50  0001 C CNN
-	1    8650 6000
-	-1   0    0    -1
-$EndComp
 $Comp
 L Device:D_Schottky D1
@@
 L power:GND #PWR0121
 U 1 1 5CC79600
-P 9050 6100
-F 0 "#PWR0121" H 9050 5850 50  0001 C CNN
-F 1 "GND" H 9055 5927 50  0000 C CNN
-F 2 "" H 9050 6100 50  0001 C CNN
-F 3 "" H 9050 6100 50  0001 C CNN
-	1    9050 6100
-	1    0    0    -1
-$EndComp
-Wire Wire Line
-	9050 6100 8850 6100
+P 8850 5800
+F 0 "#PWR0121" H 8850 5550 50  0001 C CNN
+F 1 "GND" H 8855 5627 50  0000 C CNN
+F 2 "" H 8850 5800 50  0001 C CNN
+F 3 "" H 8850 5800 50  0001 C CNN
+	1    8850 5800
+	0    -1   -1   0
+$EndComp
 $Comp
 L Connector_Generic:Conn_01x02 J?
@@
 Wire Wire Line
 	2550 5600 2700 5600
+$Comp
+L QPACE-DevelopmentBoard-rescue:Conn_01x04-conn J5
+U 1 1 5CD4F3FF
+P 8650 5800
+F 0 "J5" H 8729 5792 50  0000 L CNN
+F 1 "RPi_COMPort" H 8729 5701 50  0000 L CNN
+F 2 "Socket_Strips:Socket_Strip_Straight_1x04_Pitch2.54mm" H 8650 5800 50  0001 C CNN
+F 3 "~" H 8650 5800 50  0001 C CNN
+	1    8650 5800
+	-1   0    0    -1
+$EndComp
+$Comp
+L power:+5V #PWR0119
+U 1 1 5CD53BAC
+P 8850 5700
+F 0 "#PWR0119" H 8850 5550 50  0001 C CNN
+F 1 "+5V" H 8865 5873 50  0000 C CNN
+F 2 "" H 8850 5700 50  0001 C CNN
+F 3 "" H 8850 5700 50  0001 C CNN
+	1    8850 5700
+	-1   0    0    -1
+$EndComp
 $EndSCHEMATC

Commit message: ready for production
passed all KiCad error checking. schematic and pcblayout were both validated. ready to be ordered
Parts:
- removed D2, D3: D_Schottky, project_footprints:SOD-128, symbol Device:D_Schottky
- added J11: RF_External_Sim, Socket_Strips:Socket_Strip_Straight_1x04_Pitch2.54mm, symbol QPACE-DevelopmentBoard-rescue:Conn_01x04-conn
- added SW1: SW_DPDT_x2, project_footprints:Pin_Header_Straight_2x03_Pitch2.54mm, symbol Switch:SW_DPDT_x2
- added TP-GND1, TP10, TP11, TP12, TP3, TP6, TP7, TP8, TP9: TestPoint, Measurement_Points:Measurement_Point_Round-SMD-Pad_Small, symbol Connector:TestPoint
- J1: footprint TerminalBlocks_Phoenix:TerminalBlock_Phoenix_PT-3.5mm_2pol -> TerminalBlocks_Phoenix:TerminalBlock_Phoenix_PT-3.5mm_3pol
- renumbered J13 to J10, J5 to J12, J7 to J5, J8 to J6, J6 to J7, J9 to J8, J10 to J9, R2 to R1, R3 to R2, R1 to R3, TP3 to TP4, TP4 to TP5
Connections:
- net +3V3: no longer U1.1 (NC)
- net +5V: now also J2.1 (Pin_1), J5.1 (Pin_1), J11.1 (Pin_1)
- net GND: now also U1.1 (NC), J11.2 (Pin_2), TP-GND1.1
- net I2C_SCL: now also TP2.1
- net I2C_SDA: now also TP3.1
- net Simluate-WTC/CCDR_UART_RX: now also TP12.1
- net Simluate-WTC/CCDR_UART_TX: now also TP11.1
- net UART_RX_CCDR: now also TP10.1
- net UART_RX_RF_int: now also SW1.5 (B), TP8.1; no longer J10.4 (Pin_4)
- net UART_TX_CCDR: now also TP9.1
- net UART_TX_RF_int: now also SW1.2 (B), TP7.1; no longer J10.3 (Pin_3)
- net at U1.4 (INT1): now also TP6.1
- new net: J10.3 (Pin_3), SW1.1 (A)
- new net: J10.4 (Pin_4), SW1.4 (A)
- new net: J11.3 (Pin_3), SW1.3 (C)
- new net: J11.4 (Pin_4), SW1.6 (C)
- no-connect marks 4 -> 3
Other:
- note added: "CCDR"
- note added: "EnduroSat RF"
- note added: "GPS"
- note added: "Gyroscope"
- note added: "Override switch for Pi power"
- note added: "Power System"
- note added: "RF"
- note added: "SWD STM32 Programmer (WTC)"
- note added: "WTC"
- moved on the sheet: C1, C2, J10, J4, J6, J7, J8, J9, R1, R2, TP4, TP5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
