File: Development Board/QPACE-DevelopmentBoard.kicad_pcb (KiCad board)
At the start: 4 copper layers, 65 x 56 mm, 61 parts, among them J1 Barrel_Jack_Switch, J10 SWD_ext, J11 Pi_I2C-BUS, J12 USB-Serial, J13 RF_External, J14 40HAT, J2 5Vin-USB, J3 Vin, J4 Vin, J6 WTC_I2C-BUS, J7 Vout, J8 Vout, J9 GPS, Q1 BSS138, Q2 Q_PMOS_GDSD, SW2 SW_SPDT, U1 BMG160, U2 SC16IS740, U3 STM32L151VETx, Y1 1.8432MHz

Commit message: added silk screen, organized pins
Parts:
- removed J12: USB-Serial, Socket_Strips:Socket_Strip_Straight_1x03_Pitch2.54mm
- added J5: RPi_COMPort, Socket_Strips:Socket_Strip_Straight_1x04_Pitch2.54mm, F.Cu at (141.6, 81.3)
Connections:
- J11 pad 1: /Simulate-CCDR/Pi_I2C_SCL -> /Simulate-CCDR/Pi_I2C_SDA
- J11 pad 2: /Simulate-CCDR/Pi_I2C_SDA -> /Simulate-CCDR/Pi_I2C_SCL
Routing:
- net +5V: track 173.5 -> 212.7 mm
- net GND: track 114.7 -> 98.3 mm, vias 19 -> 20
- net /UART_RX_CCDR: track 63.2 -> 71.6 mm, vias 0 -> 1
- net 3_3V_Rail: track 195.3 -> 200.3 mm
- net /UART_TX_CCDR: track 61.3 -> 65.3 mm
- net /Simulate-CCDR/Pi_I2C_SDA: track 60.4 -> 62.9 mm
- net /Simulate-CCDR/Pi_I2C_SCL: track 59.3 -> 57.1 mm
Other:
- outline, holes or cut-outs redrawn
- board text added: "DC-DC 5/20V to 3.3V"
- board text added: "DC-DC 5V to 3.3V"
- board text added: "Enable Pi Override (SPDT)"
- board text added: "I2C Buses STM32 & RPi"
- board text added: "Raspberry Pi Hat"
- board text added: "STM32 SWD & GPS (Secondary UART)"
- board text added: "Serial Ports RPi & RF"
- board text added: "Vin (5-20V)"
- board text added: "Vusb (5V)"

Commit message: fixed silk screen
Other:
- board text added: "DC-DC 5/20V to 5V"
- board text removed: "DC-DC 5/20V to 3.3V"
Changed lines of the file:
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@@
   )
   (setup
-    (last_trace_width 0.4)
+    (last_trace_width 0.15)
     (user_trace_width 0.15)
     (user_trace_width 0.2)
@@
     (effects (font (size 0.75 0.75) (thickness 0.1875)) (justify left mirror))
   )
-  (gr_text "DC-DC 5/20V to 3.3V" (at 99.06 101.6) (layer B.SilkS)
+  (gr_text "DC-DC 5/20V to 5V" (at 99.06 101.6) (layer B.SilkS)
     (effects (font (size 0.75 0.75) (thickness 0.1875)) (justify mirror))
   )
@@
   (segment (start 104.14 85.09) (end 104.14 101.6) (width 1) (layer B.Cu) (net 1))
   (segment (start 104.14 101.6) (end 100.33 105.41) (width 1) (layer B.Cu) (net 1))
+  (segment (start 142.113 83.312) (end 141.605 83.82) (width 0.25) (layer B.Cu) (net 1))
+  (segment (start 130.8675 75.575) (end 130.8675 76.1425) (width 0.25) (layer F.Cu) (net 1))
+  (segment (start 130.048 75.946) (end 130.302 76.2) (width 0.25) (layer B.Cu) (net 1))
+  (segment (start 130.527158 76.2) (end 130.81 76.2) (width 0.25) (layer B.Cu) (net 1))
+  (segment (start 131 76.39) (end 130.81 76.2) (width 0.25) (layer F.Cu) (net 1))
+  (segment (start 130.302 76.2) (end 130.527158 76.2) (width 0.25) (layer B.Cu) (net 1))
+  (segment (start 130.8675 76.1425) (end 130.81 76.2) (width 0.25) (layer F.Cu) (net 1))
+  (segment (start 130.048 73.66) (end 130.048 75.946) (width 0.25) (layer B.Cu) (net 1))
+  (segment (start 131 78) (end 131 76.39) (width 0.25) (layer F.Cu) (net 1))
+  (via (at 130.81 76.2) (size 0.4) (drill 0.2) (layers F.Cu B.Cu) (net 1))
+  (via (at 129.032 78.232) (size 0.4) (drill 0.2) (layers F.Cu B.Cu) (net 1))
+  (segment (start 128.524 77) (end 128.524 77.724) (width 0.4) (layer F.Cu) (net 1))
+  (segment (start 128.524 77.724) (end 129.032 78.232) (width 0.4) (layer F.Cu) (net 1))
   (segment (start 112.03 88.646) (end 112.03 90.678) (width 0.5) (layer F.Cu) (net 2) (status 30))
   (segment (start 112.03 92.198) (end 112.014 92.214) (width 0.5) (layer F.Cu) (net 2) (status 30))
@@
   (segment (start 112.776 83.82) (end 112.776 82.458946) (width 0.25) (layer F.Cu) (net 2) (status 10))
   (segment (start 112.776 82.458946) (end 112.395 82.077946) (width 0.25) (layer F.Cu) (net 2))
+  (segment (start 128.599 75.075) (end 128.524 75) (width 0.25) (layer F.Cu) (net 2))
+  (segment (start 130.8675 75.075) (end 128.599 75.075) (width 0.25) (layer F.Cu) (net 2))
+  (segment (start 129.794 76.145) (end 129.794 79.248) (width 0.4) (layer F.Cu) (net 2))
+  (segment (start 128.649 75) (end 129.794 76.145) (width 0.4) (layer F.Cu) (net 2))
+  (segment (start 128.524 75) (end 128.649 75) (width 0.4) (layer F.Cu) (net 2))
+  (segment (start 134.366 77.534) (end 134.366 75.438) (width 0.4) (layer F.Cu) (net 2))
+  (segment (start 133.9 78) (end 134.366 77.534) (width 0.4) (layer F.Cu) (net 2))
+  (segment (start 133 78) (end 133.9 78) (width 0.4) (layer F.Cu) (net 2))
   (segment (start 122.825 73.93) (end 120.65 73.93) (width 0.25) (layer F.Cu) (net 3) (status 20))
   (segment (start 124.46 75.565) (end 122.825 73.93) (width 0.25) (layer F.Cu) (net 3) (status 10))
@@
   (segment (start 106.934 97.536) (end 121.666 112.268) (width 1) (layer F.Cu) (net 8))
   (segment (start 139.065 81.28) (end 102.362 81.28) (width 1) (layer B.Cu) (net 8) (status 10))
+  (segment (start 141.605 81.28) (end 139.065 81.28) (width 1) (layer F.Cu) (net 8))
   (segment (start 87.632 88.052) (end 84.582 88.052) (width 2) (layer F.Cu) (net 9) (status 20))
   (segment (start 99.68 88.052) (end 87.632 88.052) (width 2) (layer F.Cu) (net 9))
@@
   (segment (start 134.804992 85.27499) (end 134.960001 85.429999) (width 0.25) (layer F.Cu) (net 17))
   (segment (start 133.02699 85.27499) (end 134.804992 85.27499) (width 0.25) (layer F.Cu) (net 17))
-  (segment (start 142.113 83.312) (end 141.605 83.82) (width 0.25) (layer B.Cu) (net 1))
-  (segment (start 130.8675 75.575) (end 130.8675 76.1425) (width 0.25) (layer F.Cu) (net 1))
-  (segment (start 130.048 75.946) (end 130.302 76.2) (width 0.25) (layer B.Cu) (net 1))
-  (segment (start 130.527158 76.2) (end 130.81 76.2) (width 0.25) (layer B.Cu) (net 1))
-  (segment (start 131 76.39) (end 130.81 76.2) (width 0.25) (layer F.Cu) (net 1))
-  (segment (start 130.302 76.2) (end 130.527158 76.2) (width 0.25) (layer B.Cu) (net 1))
-  (segment (start 130.8675 76.1425) (end 130.81 76.2) (width 0.25) (layer F.Cu) (net 1))
-  (segment (start 130.048 73.66) (end 130.048 75.946) (width 0.25) (layer B.Cu) (net 1))
-  (segment (start 131 78) (end 131 76.39) (width 0.25) (layer F.Cu) (net 1))
-  (via (at 130.81 76.2) (size 0.4) (drill 0.2) (layers F.Cu B.Cu) (net 1))
-  (via (at 129.032 78.232) (size 0.4) (drill 0.2) (layers F.Cu B.Cu) (net 1))
-  (segment (start 128.524 77) (end 128.524 77.724) (width 0.4) (layer F.Cu) (net 1))
-  (segment (start 128.524 77.724) (end 129.032 78.232) (width 0.4) (layer F.Cu) (net 1))
-  (segment (start 128.599 75.075) (end 128.524 75) (width 0.25) (layer F.Cu) (net 2))
-  (segment (start 130.8675 75.075) (end 128.599 75.075) (width 0.25) (layer F.Cu) (net 2))
-  (segment (start 129.794 76.145) (end 129.794 79.248) (width 0.4) (layer F.Cu) (net 2))
-  (segment (start 128.649 75) (end 129.794 76.145) (width 0.4) (layer F.Cu) (net 2))
-  (segment (start 128.524 75) (end 128.649 75) (width 0.4) (layer F.Cu) (net 2))
-  (segment (start 134.366 77.534) (end 134.366 75.438) (width 0.4) (layer F.Cu) (net 2))
-  (segment (start 133.9 78) (end 134.366 77.534) (width 0.4) (layer F.Cu) (net 2))
-  (segment (start 133 78) (end 133.9 78) (width 0.4) (layer F.Cu) (net 2))
-  (segment (start 141.605 81.28) (end 139.065 81.28) (width 1) (layer F.Cu) (net 8))
   (segment (start 136.652 69.975589) (end 136.652 76.962) (width 0.25) (layer B.Cu) (net 18))
   (segment (start 104.313631 68.112988) (end 134.789399 68.112988) (width 0.25) (layer B.Cu) (net 18))

Commit message: ready for production
passed all KiCad error checking. schematic and pcblayout were both validated. ready to be ordered
Parts:
- removed D2, D3: D_Schottky, project_footprints:SOD-128
- added SW1: SW_DPDT_x2, project_footprints:Pin_Header_Straight_2x03_Pitch2.54mm, F.Cu at (125.7, 114.9)
- added TP-GND1: TestPoint, Measurement_Points:Measurement_Point_Round-SMD-Pad_Small, F.Cu at (81.5, 81.8)
- added TP10: TestPoint, Measurement_Points:Measurement_Point_Round-SMD-Pad_Small, F.Cu at (139.1, 88.9)
- added TP11: TestPoint, Measurement_Points:Measurement_Point_Round-SMD-Pad_Small, F.Cu at (119.9, 82.8)
- added TP12: TestPoint, Measurement_Points:Measurement_Point_Round-SMD-Pad_Small, F.Cu at (119.9, 80.8)
- added TP15: TestPoint, Measurement_Points:Measurement_Point_Round-SMD-Pad_Small, F.Cu at (107.2, 71.6)
- added TP16: TestPoint, Measurement_Points:Measurement_Point_Round-SMD-Pad_Small, F.Cu at (107.7, 69.6)
- added TP3: TestPoint, Measurement_Points:Measurement_Point_Round-SMD-Pad_Small, F.Cu at (139.2, 71.1)
- added TP6: TestPoint, Measurement_Points:Measurement_Point_Round-SMD-Pad_Small, F.Cu at (136.7, 73.9)
- added TP7: TestPoint, Measurement_Points:Measurement_Point_Round-SMD-Pad_Small, F.Cu at (134.0, 114.9)
- added TP8: TestPoint, Measurement_Points:Measurement_Point_Round-SMD-Pad_Small, F.Cu at (134.0, 112.4)
- added TP9: TestPoint, Measurement_Points:Measurement_Point_Round-SMD-Pad_Small, F.Cu at (139.1, 86.4)
- J1: footprint TerminalBlocks_Phoenix:TerminalBlock_Phoenix_PT-3.5mm_2pol -> TerminalBlocks_Phoenix:TerminalBlock_Phoenix_PT-3.5mm_3pol
- J11: value Pi_I2C-BUS -> RF_External_Sim; footprint Socket_Strips:Socket_Strip_Straight_1x03_Pitch2.54mm -> Socket_Strips:Socket_Strip_Straight_1x04_Pitch2.54mm
- R13, R14: value 10k -> 4.99K
- moved TP2 56.5 mm to (139.2, 73.7)
- moved J11 48.6 mm to (113.0, 112.4), turned to 90 degrees
- moved J10 42.5 mm to (113.0, 114.9), turned to 90 degrees
- moved J3 14.5 mm to (89.7, 109.2), turned to 180 degrees
- moved J4 14.5 mm to (89.7, 92.2), turned to 180 degrees
- moved J5 14.5 mm to (109.2, 109.2), turned to 180 degrees
- moved J6 14.5 mm to (109.2, 92.2), turned to 180 degrees
- moved TP5 7.64 mm to (86.9, 87.9)
- moved D1 5.59 mm to (83.1, 92.2)
- moved J2 5.59 mm to (81.3, 85.9)
- moved J1 3.36 mm to (83.8, 100.6)
- moved TP1 3.14 mm to (87.1, 97.8)
- renumbered J13 to J10, J5 to J12, J14 to J13, J7 to J5, J8 to J6, J6 to J7, J9 to J8, J10 to J9, R2 to R1, R3 to R2, R1 to R3, TP5 to TP13, TP6 to TP14, TP7 to TP17, TP3 to TP4, TP4 to TP5
Connections:
- J10 pad 3: /UART_TX_RF_int -> Net-(J10-Pad3)
- J10 pad 4: /UART_RX_RF_int -> Net-(J10-Pad4)
- J11 pad 1: /Simulate-CCDR/Pi_I2C_SDA -> +5V
- J11 pad 2: /Simulate-CCDR/Pi_I2C_SCL -> GND
- J11 pad 3: GND -> Net-(J11-Pad3)
- J13 pad 12: (no net) -> /PiHeartBeat
- J2 pad 1: Net-(D3-Pad2) -> +5V
- J5 pad 1: Net-(D2-Pad2) -> +5V
- TP2 pad 1: Net-(D3-Pad2) -> /I2C_SCL
- U1 pad 1: 3_3V_Rail -> GND
- U1 pad 4: (no net) -> Net-(TP6-Pad1)
- U3 pad 21: GND -> 3_3V_Rail
- U3 pad 25: /GPS_TX -> /GPS_RX
- U3 pad 26: /GPS_RX -> /GPS_TX
- U3 pad 47: /I2C_SDA -> /I2C_SCL
- U3 pad 48: /I2C_SCL -> /I2C_SDA
- U3 pad 58: (no net) -> /En_PiPwr
- U3 pad 62: (no net) -> /PiHeartBeat
Routing:
- net GND: track 98.3 -> 206.2 mm, vias 20 -> 44
- net /En_PiPwr: track 17.7 -> 81.3 mm, vias 0 -> 2
- net /PiHeartBeat: track 0.00 -> 63.4 mm, vias 0 -> 5
- net /Simulate-CCDR/Pi_I2C_SDA: track 62.9 -> 29.9 mm
- net /Simulate-CCDR/Pi_I2C_SCL: track 57.1 -> 28.0 mm
- net Net-(D2-Pad2): track 27.4 -> 0.00 mm
- net /UART_TX_RF_int: track 11.5 -> 34.6 mm
- net /UART_RX_RF_int: track 11.0 -> 30.8 mm
- net Net-(J11-Pad3): track 0.00 -> 13.8 mm
- net Net-(D1-Pad1): track 5.67 -> 18.8 mm
- net Net-(J11-Pad4): track 0.00 -> 11.2 mm
- net 3_3V_Rail: track 200.3 -> 211.2 mm
- net Net-(J10-Pad3): track 0.00 -> 8.59 mm
- net Net-(D3-Pad2): track 8.28 -> 0.00 mm
- net +5V: track 212.7 -> 206.4 mm, vias 5 -> 6
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Other:
- outline, holes or cut-outs redrawn
- board text added: "CCDR/Pi"
- board text added: "Enable Pi Override"
- board text added: "GYRO"
- board text added: "Q-PACE Development Board Raspiberry Pi Hat V0 / by TCC"
- board text added: "RF switch"
- board text added: "RPi COM Port"
- board text added: "SWD GPS"
- board text added: "Vin: 5-20V Vout: 5V"
- board text added: "Vin: 5V Vout: 3.3V"
- board text added: "WTC"
- board text added: "WTC I2C Bus"
- board text added: "WTC-CCDR COMMS"
- board text added: "sim RF real RF"
- board text removed: "Enable Pi Override (SPDT)"
- board text removed: "I2C Buses STM32 & RPi"
- board text removed: "Q-PACE Development Board V0 / TCC"
- board text removed: "Raspberry Pi Hat"
- board text removed: "Serial Ports RPi & RF"

Commit message: fix
Other:
- board text added: "GPS SWD"
- board text removed: "SWD GPS"
Changed lines of the file:
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@@
     )
+  )
+  (gr_text "GPS SWD" (at 137.668 91.44) (layer F.SilkS)
+    (effects (font (size 0.75 0.75) (thickness 0.1875)) (justify left))
   )
   (gr_text CCDR/Pi (at 85.852 68.072) (layer F.SilkS)
@@
     (effects (font (size 0.75 0.75) (thickness 0.1875)) (justify right))
   )
-  (gr_text "SWD GPS" (at 137.668 108.712) (layer F.SilkS)
+  (gr_text "GPS SWD" (at 137.668 108.712) (layer F.SilkS)
     (effects (font (size 0.75 0.75) (thickness 0.1875)) (justify left))
   )
-  (gr_text "SWD GPS" (at 137.668 91.44) (layer F.SilkS)
-    (effects (font (size 0.75 0.75) (thickness 0.1875)) (justify left))
-  )
